File: Hardware/SmartNode/mainbrd.sch (EAGLE design)
At the start: 42 parts, among them U1 NRF51822-QFAA, U2 CC3000, X1 87438-06, Y1 16MHz, Y2 32.768kHz

Commit message: Updated Hardware Files
Parts:
- removed R3: NL, rcl:R-US_R0402
- U$2: value AT8010 -> PCB_ANT; device SmartNodeLib:AT8010 -> SmartNodeLib:PCB_ANT
Connections:
- removed net N$11: C15.1, C6.1, L3.1, U$2.FP
- new net ANT: C15.1, C6.1, L3.1, U$2.P$1
- net GND: no longer R3.1
- net N$16: now also U1.P0.29; no longer U1.P0.21
- net N$19: no longer R3.2
- net SPI_CLK: now also U1.P0.01/AIN2; no longer U1.P0.22
- net SPI_CS: now also U1.P0.05/AIN6; no longer U1.P0.23
- net SPI_IRQ: now also U1.P0.03/AIN4; no longer U1.P0.28
- net SPI_MISO: now also U1.P0.04/AIN5; no longer U1.P0.25
- net SPI_MOSI: now also U1.P0.02/AIN3; no longer U1.P0.24
- net UART_RX: now also U1.P0.15, X1-5.S; no longer U1.P0.16, X1-4.S
- net UART_TX: now also U1.P0.16, X1-4.S; no longer U1.P0.15, X1-5.S
- net VBAT_SW_EN: now also U1.P0.00/AREF0; no longer U1.P0.29
Other:
- note removed: "Load R3 and remove R4 for Testing"
- moved on the sheet: C12, C7, L4, L5, LED1, R2, R4, X1-1, X1-2, X1-3, X1-4, X1-5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

Commit message: sync everything up
Parts:
- removed X1: 87438-06, con-molex:87438-06
- added P1, P2: FTSH-105-01-L-DV-K, con-samtec:FTSH-105-01-L-DV-K
Connections:
- net GND: now also P1.3, P1.5, P1.9, P2.3, P2.5, P2.9; no longer X1-1.S
- net SWDCLK: now also P1.4; no longer X1-2.S
- net SWDIO: now also P1.2; no longer X1-3.S
- net UART_RX: now also P2.2; no longer X1-5.S
- net UART_TX: now also P2.4; no longer X1-4.S
- net VCC: now also P1.1, P2.1; no longer X1-6.S
